File: stereo_amp/stereo_amp.sch (KiCad schematic (older format))
At the start: 31 parts, among them K1 CONN_3, P1 CONN_3X2, P2 CONN_1, P3 CONN_1, P4 CONN_1, P5 CONN_1, P6 CONN_1, P7 CONN_1, P8 CONN_1, Q1 TIP41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

Commit message: Started on bike speedometer/computer thing
Parts:
- gave numbers to parts that had none: 2
Changed lines of the file:
@@
-EESchema Schematic File Version 2  date Sat 19 Apr 2014 05:49:17 PM CEST
+EESchema Schematic File Version 2  date Sat 19 Apr 2014 09:20:30 PM CEST
 LIBS:power
 LIBS:device
@@
 	3200 2050 3200 2200
 $Comp
-L -12V #PWR?
+L -12V #PWR01
 U 1 1 53529AF2
 P 3200 2750
-F 0 "#PWR?" H 3200 2880 20  0001 C CNN
+F 0 "#PWR01" H 3200 2880 20  0001 C CNN
 F 1 "-12V" H 3200 2850 30  0000 C CNN
 	1    3200 2750
@@
 $EndComp
 $Comp
-L +12V #PWR?
+L +12V #PWR02
 U 1 1 53529AD4
 P 3200 2050
-F 0 "#PWR?" H 3200 2000 20  0001 C CNN
+F 0 "#PWR02" H 3200 2000 20  0001 C CNN
 F 1 "+12V" H 3200 2150 30  0000 C CNN
 	1    3200 2050
@@
 $EndComp
 $Comp
-L C C?
+L C C12
 U 1 1 53529AC5
 P 3400 2400
-F 0 "C?" H 3450 2500 50  0000 L CNN
+F 0 "C12" H 3450 2500 50  0000 L CNN
 F 1 "C" H 3450 2300 50  0000 L CNN
 	1    3400 2400
@@
 $EndComp
 $Comp
-L C C?
+L C C11
 U 1 1 53529AC1
 P 3000 2400
-F 0 "C?" H 3050 2500 50  0000 L CNN
+F 0 "C11" H 3050 2500 50  0000 L CNN
 F 1 "C" H 3050 2300 50  0000 L CNN
 	1    3000 2400
@@
 $EndComp
 $Comp
-L GND #PWR18
+L GND #PWR03
 U 1 1 53528B6D
 P 7950 4400
-F 0 "#PWR18" H 7950 4400 30  0001 C CNN
+F 0 "#PWR03" H 7950 4400 30  0001 C CNN
 F 1 "GND" H 7950 4330 30  0001 C CNN
 	1    7950 4400
@@
 $EndComp
 $Comp
-L +12V #PWR19
+L +12V #PWR04
 U 1 1 53528B5C
 P 8200 4000
-F 0 "#PWR19" H 8200 3950 20  0001 C CNN
+F 0 "#PWR04" H 8200 3950 20  0001 C CNN
 F 1 "+12V" H 8200 4100 30  0000 C CNN
 	1    8200 4000
@@
 $EndComp
 $Comp
-L -12V #PWR20
+L -12V #PWR05
 U 1 1 53528B54
 P 8200 4800
-F 0 "#PWR20" H 8200 4930 20  0001 C CNN
+F 0 "#PWR05" H 8200 4930 20  0001 C CNN
 F 1 "-12V" H 8200 4900 30  0000 C CNN
 	1    8200 4800
@@
 $EndComp
 $Comp
-L GND #PWR17
+L GND #PWR06
 U 1 1 53528B1A
 P 7750 5650
-F 0 "#PWR17" H 7750 5650 30  0001 C CNN
+F 0 "#PWR06" H 7750 5650 30  0001 C CNN
 F 1 "GND" H 7750 5580 30  0001 C CNN
 	1    7750 5650
@@
 $EndComp
 $Comp
-L GND #PWR16
+L GND #PWR07
 U 1 1 53528ABD
 P 7750 3150
-F 0 "#PWR16" H 7750 3150 30  0001 C CNN
+F 0 "#PWR07" H 7750 3150 30  0001 C CNN
 F 1 "GND" H 7750 3080 30  0001 C CNN
 	1    7750 3150
@@
 $EndComp
 $Comp
-L -12V #PWR15
+L -12V #PWR08
 U 1 1 53528A4B
 P 7400 6050
-F 0 "#PWR15" H 7400 6180 20  0001 C CNN
+F 0 "#PWR08" H 7400 6180 20  0001 C CNN
 F 1 "-12V" H 7400 6150 30  0000 C CNN
 	1    7400 6050
@@
 $EndComp
 $Comp
-L -12V #PWR13
+L -12V #PWR09
 U 1 1 53528986
 P 7400 4150
-F 0 "#PWR13" H 7400 4280 20  0001 C CNN
+F 0 "#PWR09" H 7400 4280 20  0001 C CNN
 F 1 "-12V" H 7400 4250 30  0000 C CNN
 	1    7400 4150
@@
 $EndComp
 $Comp
-L +12V #PWR14
+L +12V #PWR010
 U 1 1 5352891E
 P 7400 4650
-F 0 "#PWR14" H 7400 4600 20  0001 C CNN
+F 0 "#PWR010" H 7400 4600 20  0001 C CNN
 F 1 "+12V" H 7400 4750 30  0000 C CNN
 	1    7400 4650
@@
 $EndComp
 $Comp
-L +12V #PWR12
+L +12V #PWR011
 U 1 1 535288ED
 P 7400 2750
-F 0 "#PWR12" H 7400 2700 20  0001 C CNN
+F 0 "#PWR011" H 7400 2700 20  0001 C CNN
 F 1 "+12V" H 7400 2850 30  0000 C CNN
 	1    7400 2750
@@
 $EndComp
 $Comp
-L -12V #PWR9
+L -12V #PWR012
 U 1 1 535287EC
 P 6200 3950
-F 0 "#PWR9" H 6200 4080 20  0001 C CNN
+F 0 "#PWR012" H 6200 4080 20  0001 C CNN
 F 1 "-12V" H 6200 4050 30  0000 C CNN
 	1    6200 3950
@@
 $EndComp
 $Comp
-L -12V #PWR10
+L -12V #PWR013
 U 1 1 535287E7
 P 6200 4850
-F 0 "#PWR10" H 6200 4980 20  0001 C CNN
+F 0 "#PWR013" H 6200 4980 20  0001 C CNN
 F 1 "-12V" H 6200 4950 30  0000 C CNN
 	1    6200 4850
@@
 $EndComp
 $Comp
-L +12V #PWR11
+L +12V #PWR014
 U 1 1 535287D6
 P 6200 5850
-F 0 "#PWR11" H 6200 5800 20  0001 C CNN
+F 0 "#PWR014" H 6200 5800 20  0001 C CNN
 F 1 "+12V" H 6200 5950 30  0000 C CNN
 	1    6200 5850
@@
 $EndComp
 $Comp
-L +12V #PWR8
+L +12V #PWR015
 U 1 1 535287C6
 P 6200 2950
-F 0 "#PWR8" H 6200 2900 20  0001 C CNN
+F 0 "#PWR015" H 6200 2900 20  0001 C CNN
 F 1 "+12V" H 6200 3050 30  0000 C CNN
 	1    6200 2950
@@
 $EndComp
 $Comp
-L GND #PWR7
+L GND #PWR016
 U 1 1 5352874D
 P 5700 5550
-F 0 "#PWR7" H 5700 5550 30  0001 C CNN
+F 0 "#PWR016" H 5700 5550 30  0001 C CNN
 F 1 "GND" H 5700 5480 30  0001 C CNN
 	1    5700 5550
@@
 $EndComp
 $Comp
-L GND #PWR6
+L GND #PWR017
 U 1 1 53528735
 P 5700 3250
-F 0 "#PWR6" H 5700 3250 30  0001 C CNN
+F 0 "#PWR017" H 5700 3250 30  0001 C CNN
 F 1 "GND" H 5700 3180 30  0001 C CNN
 	1    5700 3250
@@
 VOLUME
 $Comp
-L -12V #PWR5
+L -12V #PWR018
 U 1 1 535286A0
 P 4650 5850
-F 0 "#PWR5" H 4650 5980 20  0001 C CNN
+F 0 "#PWR018" H 4650 5980 20  0001 C CNN
 F 1 "-12V" H 4650 5950 30  0000 C CNN
 	1    4650 5850
@@
 $EndComp
 $Comp
-L -12V #PWR2
+L -12V #PWR019
 U 1 1 5352869C
 P 4650 2950
-F 0 "#PWR2" H 4650 3080 20  0001 C CNN
+F 0 "#PWR019" H 4650 3080 20  0001 C CNN
 F 1 "-12V" H 4650 3050 30  0000 C CNN
 	1    4650 2950
@@
 $EndComp
 $Comp
-L +12V #PWR4
+L +12V #PWR020
 U 1 1 53528692
 P 4650 4850
-F 0 "#PWR4" H 4650 4800 20  0001 C CNN
+F 0 "#PWR020" H 4650 4800 20  0001 C CNN
 F 1 "+12V" H 4650 4950 30  0000 C CNN
 	1    4650 4850
@@
 $EndComp
 $Comp
-L +12V #PWR3
+L +12V #PWR021
 U 1 1 5352868E
 P 4650 3950
-F 0 "#PWR3" H 4650 3900 20  0001 C CNN
+F 0 "#PWR021" H 4650 3900 20  0001 C CNN
 F 1 "+12V" H 4650 4050 30  0000 C CNN
 	1    4650 3950
@@
 $EndComp
 $Comp
-L GND #PWR1
+L GND #PWR022
 U 1 1 53528557
 P 4050 4400
-F 0 "#PWR1" H 4050 4400 30  0001 C CNN
+F 0 "#PWR022" H 4050 4400 30  0001 C CNN
 F 1 "GND" H 4050 4330 30  0001 C CNN
 	1    4050 4400
