File: bike_computer/bikomp.sch (KiCad schematic (older format))
At the start: 10 parts, among them P1 CONN_8, U1 HD44780, U2 74LS154, U3 2716, U4 M6809P, U5 74LS374, U6 74LS374

Commit message: Schematic more or less done
Parts:
- added C1, C2: 27 pF, symbol C
- added C3: CP1, symbol CP1
- added P2: CONN_1, symbol CONN_1
- added RV1: POT, symbol POT
- added U7: 40106, symbol 40106
- added U8: 74LS109, symbol 74LS109
- added U9: 96LC48, symbol 96LC48
- added X1: CRYSTAL, symbol CRYSTAL
Connections:
- net labels added: CLEAR_INT, EE_SEL, RAM_OE, SPI_SSEL0, VDD, VSS
- wire segments 131 -> 187

Commit message: Decoupling
Parts:
- added C10, C4, C5, C6, C7, C8, C9: C, symbol C
Connections:
- wire segments 187 -> 191

Commit message: Fixed some derps
Parts:
- added R2, R3: 10 kΩ, symbol R
Connections:
- wire segments 191 -> 194
Changed lines of the file:
@@
-EESchema Schematic File Version 2  date Sun 25 May 2014 11:33:41 PM CEST
+EESchema Schematic File Version 2  date Mon 26 May 2014 08:21:45 PM CEST
 LIBS:power
 LIBS:device
@@
 Sheet 1 1
 Title ""
-Date "25 may 2014"
+Date "26 may 2014"
 Rev ""
 Comp ""
@@
 Comment4 ""
 $EndDescr
+Connection ~ 9300 1450
+Wire Wire Line
+	9300 1300 9300 1450
+Connection ~ 6350 1850
+Wire Wire Line
+	6350 1850 6350 1950
+Wire Wire Line
+	10850 6300 10850 6250
 Wire Wire Line
 	10100 2050 10100 1850
@@
 	4250 7100 4200 7100
 Wire Wire Line
-	10850 6850 10850 6950
-Wire Wire Line
 	9800 6800 10350 6800
 Wire Wire Line
@@
 	8000 1250 7800 1250
 Wire Wire Line
-	6350 2150 6350 1950
-Wire Wire Line
 	6350 1950 6400 1950
 Wire Wire Line
@@
 	8100 2450 5300 2450
 Wire Wire Line
-	6250 3900 6400 3900
-Wire Wire Line
 	6250 1850 6400 1850
 Wire Wire Line
@@
 	8200 5650 8200 4650
 Wire Wire Line
-	10850 6950 9800 6950
+	9800 6950 10850 6950
 Wire Wire Line
 	4000 7100 3850 7100
@@
 	10850 1850 9100 1850
 Connection ~ 10600 1850
+Wire Wire Line
+	10850 6950 10850 6800
+Wire Wire Line
+	6400 4250 6400 3900
+Wire Wire Line
+	8800 1300 8650 1300
+Connection ~ 8650 1300
+$Comp
+L R R3
+U 1 1 538382CE
+P 9050 1300
+F 0 "R3" V 9130 1300 50  0000 C CNN
+F 1 "10 kΩ" V 9050 1300 50  0000 C CNN
+	1    9050 1300
+	0    -1   -1   0
+$EndComp
 $Comp
 L GND #PWR01
+U 1 1 5383806A
+P 6400 4250
+F 0 "#PWR01" H 6400 4250 30  0001 C CNN
+F 1 "GND" H 6400 4180 30  0001 C CNN
+	1    6400 4250
+	1    0    0    -1
+$EndComp
+$Comp
+L R R2
+U 1 1 538370E5
+P 10850 6550
+F 0 "R2" V 10930 6550 50  0000 C CNN
+F 1 "10 kΩ" V 10850 6550 50  0000 C CNN
+	1    10850 6550
+	1    0    0    -1
+$EndComp
+$Comp
+L GND #PWR02
 U 1 1 53812E12
 P 10100 2050
-F 0 "#PWR01" H 10100 2050 30  0001 C CNN
+F 0 "#PWR02" H 10100 2050 30  0001 C CNN
 F 1 "GND" H 10100 1980 30  0001 C CNN
 	1    10100 2050
@@
 $EndComp
 $Comp
-L VCC #PWR02
+L VCC #PWR03
 U 1 1 53812E09
 P 10100 1350
-F 0 "#PWR02" H 10100 1450 30  0001 C CNN
+F 0 "#PWR03" H 10100 1450 30  0001 C CNN
 F 1 "VCC" H 10100 1450 30  0000 C CNN
 	1    10100 1350
@@
 $EndComp
 $Comp
-L GND #PWR03
+L GND #PWR04
 U 1 1 5380A4FE
 P 2300 4600
-F 0 "#PWR03" H 2300 4600 30  0001 C CNN
+F 0 "#PWR04" H 2300 4600 30  0001 C CNN
 F 1 "GND" H 2300 4530 30  0001 C CNN
 	1    2300 4600
@@
 $EndComp
 $Comp
-L VCC #PWR04
+L VCC #PWR05
 U 1 1 5380A4F9
 P 2300 3950
-F 0 "#PWR04" H 2300 4050 30  0001 C CNN
+F 0 "#PWR05" H 2300 4050 30  0001 C CNN
 F 1 "VCC" H 2300 4050 30  0000 C CNN
 	1    2300 3950
@@
 $EndComp
 $Comp
-L VCC #PWR05
+L VCC #PWR06
 U 1 1 5380A110
 P 950 1700
-F 0 "#PWR05" H 950 1800 30  0001 C CNN
+F 0 "#PWR06" H 950 1800 30  0001 C CNN
 F 1 "VCC" H 950 1800 30  0000 C CNN
 	1    950  1700
@@
 $EndComp
 $Comp
-L GND #PWR06
+L GND #PWR07
 U 1 1 5380A10C
 P 700 1850
-F 0 "#PWR06" H 700 1850 30  0001 C CNN
+F 0 "#PWR07" H 700 1850 30  0001 C CNN
 F 1 "GND" H 700 1780 30  0001 C CNN
 	1    700  1850
@@
 $EndComp
 $Comp
-L GND #PWR07
+L GND #PWR08
 U 1 1 5380A0B5
 P 2500 1700
-F 0 "#PWR07" H 2500 1700 30  0001 C CNN
+F 0 "#PWR08" H 2500 1700 30  0001 C CNN
 F 1 "GND" H 2500 1630 30  0001 C CNN
 	1    2500 1700
@@
 $EndComp
 $Comp
-L VCC #PWR08
+L VCC #PWR09
 U 1 1 5380A0B1
 P 2400 1700
-F 0 "#PWR08" H 2400 1800 30  0001 C CNN
+F 0 "#PWR09" H 2400 1800 30  0001 C CNN
 F 1 "VCC" H 2400 1800 30  0000 C CNN
 	1    2400 1700
@@
 $EndComp
 $Comp
-L VDD #PWR09
+L VDD #PWR010
 U 1 1 53809F25
 P 10750 3300
-F 0 "#PWR09" H 10750 3400 30  0001 C CNN
+F 0 "#PWR010" H 10750 3400 30  0001 C CNN
 F 1 "VDD" H 10750 3410 30  0000 C CNN
 	1    10750 3300
@@
 $EndComp
 $Comp
-L VCC #PWR010
+L VCC #PWR011
 U 1 1 53809F21
 P 10750 3200
-F 0 "#PWR010" H 10750 3300 30  0001 C CNN
+F 0 "#PWR011" H 10750 3300 30  0001 C CNN
 F 1 "VCC" H 10750 3300 30  0000 C CNN
 	1    10750 3200
@@
 $EndComp
 $Comp
-L GND #PWR011
+L GND #PWR012
 U 1 1 53809F1D
 P 10550 3200
-F 0 "#PWR011" H 10550 3200 30  0001 C CNN
+F 0 "#PWR012" H 10550 3200 30  0001 C CNN
 F 1 "GND" H 10550 3130 30  0001 C CNN
 	1    10550 3200
@@
 $EndComp
 $Comp
-L VSS #PWR012
+L VSS #PWR013
 U 1 1 53809F1A
 P 10550 3300
-F 0 "#PWR012" H 10550 3300 30  0001 C CNN
+F 0 "#PWR013" H 10550 3300 30  0001 C CNN
 F 1 "VSS" H 10550 3230 30  0000 C CNN
 	1    10550 3300
@@
 FINT
 $Comp
-L VCC #PWR013
+L VCC #PWR014
 U 1 1 53809656
-P 10850 6850
-F 0 "#PWR013" H 10850 6950 30  0001 C CNN
-F 1 "VCC" H 10850 6950 30  0000 C CNN
-	1    10850 6850
+P 10850 6250
+F 0 "#PWR014" H 10850 6350 30  0001 C CNN
+F 1 "VCC" H 10850 6350 30  0000 C CNN
+	1    10850 6250
 	1    0    0    -1
 $EndComp
@@
 	9700 6700 9800 6800
 $Comp
-L GND #PWR014
+L GND #PWR015
 U 1 1 538092CF
 P 8650 6050
-F 0 "#PWR014" H 8650 6050 30  0001 C CNN
+F 0 "#PWR015" H 8650 6050 30  0001 C CNN
 F 1 "GND" H 8650 5980 30  0001 C CNN
 	1    8650 6050
@@
 	9600 6450 9700 6550
 $Comp
-L VCC #PWR015
+L VCC #PWR016
 U 1 1 53809224
 P 9600 4950
-F 0 "#PWR015" H 9600 5050 30  0001 C CNN
+F 0 "#PWR016" H 9600 5050 30  0001 C CNN
 F 1 "VCC" H 9600 5050 30  0000 C CNN
 	1    9600 4950
@@
 $EndComp
 $Comp
-L VCC #PWR016
+L VCC #PWR017
 U 1 1 53808811
 P 4000 7150
-F 0 "#PWR016" H 4000 7250 30  0001 C CNN
+F 0 "#PWR017" H 4000 7250 30  0001 C CNN
 F 1 "VCC" H 4000 7250 30  0000 C CNN
 	1    4000 7150
@@
 $EndComp
 $Comp
-L GND #PWR017
+L GND #PWR018
 U 1 1 5380880E
 P 4200 7150
-F 0 "#PWR017" H 4200 7150 30  0001 C CNN
+F 0 "#PWR018" H 4200 7150 30  0001 C CNN
 F 1 "GND" H 4200 7080 30  0001 C CNN
 	1    4200 7150
@@
 $EndComp
 $Comp
-L VCC #PWR018
+L VCC #PWR019
 U 1 1 538086E8
 P 3150 6100
-F 0 "#PWR018" H 3150 6200 30  0001 C CNN
+F 0 "#PWR019" H 3150 6200 30  0001 C CNN
 F 1 "VCC" H 3150 6200 30  0000 C CNN
 	1    3150 6100
@@
 $EndComp
 $Comp
-L GND #PWR019
+L GND #PWR020
 U 1 1 538086CF
 P 1550 6050
-F 0 "#PWR019" H 1550 6050 30  0001 C CNN
+F 0 "#PWR020" H 1550 6050 30  0001 C CNN
 F 1 "GND" H 1550 5980 30  0001 C CNN
 	1    1550 6050
@@
 $EndComp
 $Comp
-L GND #PWR020
+L GND #PWR021
 U 1 1 537FB130
 P 9100 3400
-F 0 "#PWR020" H 9100 3400 30  0001 C CNN
+F 0 "#PWR021" H 9100 3400 30  0001 C CNN
 F 1 "GND" H 9100 3330 30  0001 C CNN
 	1    9100 3400
@@
 $EndComp
 $Comp
-L VCC #PWR021
+L VCC #PWR022
 U 1 1 537FB12A
 P 9150 3500
-F 0 "#PWR021" H 9150 3600 30  0001 C CNN
+F 0 "#PWR022" H 9150 3600 30  0001 C CNN
 F 1 "VCC" H 9150 3600 30  0000 C CNN
 	1    9150 3500
@@
 Text Label 6250 2900 0    60   ~ 0
 D0
-$Comp
-L GND #PWR022
-U 1 1 537FA444
-P 6350 2150
-F 0 "#PWR022" H 6350 2150 30  0001 C CNN
-F 1 "GND" H 6350 2080 30  0001 C CNN
-	1    6350 2150
-	1    0    0    -1
-$EndComp
 Entry Wire Line
 	6150 3500 6250 3600
@@
 Entry Wire Line
 	6150 2800 6250 2900
-Text Label 6250 3900 0    60   ~ 0
-OUT_ENABLE
 Text Label 6250 3800 0    60   ~ 0
 OUT_ENABLE
@@
 Entry Wire Line
 	5200 1150 5300 1250
-Entry Wire Line
-	6150 3800 6250 3900
 $Comp
 L 74LS374 U6

Commit message: use oscillator instead of plain crystal
Parts:
- removed C1, C2: 27 pF, symbol C
- removed R2: 10 kΩ, symbol R
- removed U5: 74LS374, symbol 74LS374
- removed X1: CRYSTAL, symbol CRYSTAL
- added P3: CONN_2, symbol CONN_2
- added X1: OSC, symbol OSC
- U2: value 74LS154 -> 74HC154
- U6: value 74LS374 -> 74HC374
- U8: value 74LS109 -> 74HC109
Connections:
- wire segments 194 -> 189
Changed lines of the file:
@@
-EESchema Schematic File Version 2  date Mon 26 May 2014 08:21:45 PM CEST
+EESchema Schematic File Version 2  date Thu 19 Jun 2014 08:26:43 AM CEST
 LIBS:power
 LIBS:device
@@
 LIBS:m6809p
 LIBS:96lc48
+LIBS:osc
 LIBS:bikomp-cache
 EELAYER 25  0
@@
 Sheet 1 1
 Title ""
-Date "26 may 2014"
+Date "19 jun 2014"
 Rev ""
 Comp ""
@@
 Comment4 ""
 $EndDescr
+Wire Wire Line
+	2500 1600 2500 2000
+Wire Wire Line
+	2500 2000 2300 2000
+Wire Wire Line
+	2300 2000 2300 2300
+Wire Wire Line
+	2600 5900 3300 5900
+Wire Wire Line
+	2600 6250 2600 6100
 Connection ~ 9300 1450
 Wire Wire Line
@@
 Wire Wire Line
 	6350 1850 6350 1950
-Wire Wire Line
-	10850 6300 10850 6250
 Wire Wire Line
 	10100 2050 10100 1850
@@
 	1300 1850 2800 1850
 Wire Wire Line
-	2500 1700 2500 1600
-Wire Wire Line
 	10750 3300 10750 3200
 Connection ~ 4200 7100
@@
 Wire Wire Line
 	3150 6100 3300 6100
-Connection ~ 2300 5750
-Wire Wire Line
-	3300 5900 2550 5900
-Wire Wire Line
-	2550 5900 2550 5750
-Wire Wire Line
-	2550 5750 2100 5750
-Wire Wire Line
-	1700 6350 1700 5750
 Wire Wire Line
 	9150 3500 9300 3500
@@
 	6250 3000 6400 3000
 Wire Wire Line
-	1550 6050 1700 6050
-Connection ~ 1700 6050
-Wire Wire Line
-	3300 6000 2550 6000
-Wire Wire Line
-	2550 6000 2550 6350
-Wire Wire Line
-	2550 6350 2100 6350
-Connection ~ 2300 6350
-Wire Wire Line
 	3200 6200 3300 6200
 Connection ~ 3200 6100
@@
 Wire Wire Line
 	8200 5650 8200 4650
-Wire Wire Line
-	9800 6950 10850 6950
 Wire Wire Line
 	4000 7100 3850 7100
@@
 Connection ~ 10600 1850
 Wire Wire Line
-	10850 6950 10850 6800
-Wire Wire Line
 	6400 4250 6400 3900
 Wire Wire Line
 	8800 1300 8650 1300
 Connection ~ 8650 1300
+Wire Wire Line
+	2600 5700 2600 5550
+Wire Wire Line
+	2500 2300 2500 2150
+$Comp
+L CONN_2 P3
+U 1 1 53A269C9
+P 2400 2650
+F 0 "P3" V 2350 2650 40  0000 C CNN
+F 1 "CONN_2" V 2450 2650 40  0000 C CNN
+	1    2400 2650
+	0    1    1    0
+$EndComp
+$Comp
+L GND #PWR01
+U 1 1 53A25B10
+P 2600 6250
+F 0 "#PWR01" H 2600 6250 30  0001 C CNN
+F 1 "GND" H 2600 6180 30  0001 C CNN
+	1    2600 6250
+	1    0    0    -1
+$EndComp
+$Comp
+L VCC #PWR02
+U 1 1 53A25B0B
+P 2600 5550
+F 0 "#PWR02" H 2600 5650 30  0001 C CNN
+F 1 "VCC" H 2600 5650 30  0000 C CNN
+	1    2600 5550
+	1    0    0    -1
+$EndComp
+$Comp
+L OSC X1
+U 1 1 53A25AE2
+P 2150 5900
+F 0 "X1" H 2350 5800 60  0000 C CNN
+F 1 "OSC" H 2350 6000 60  0000 C CNN
+	1    2150 5900
+	-1   0    0    1
+$EndComp
+Text Label 6400 1250 0    60   ~ 0
+FINT
 $Comp
 L R R3
@@
 $EndComp
 $Comp
-L GND #PWR01
+L GND #PWR03
 U 1 1 5383806A
 P 6400 4250
-F 0 "#PWR01" H 6400 4250 30  0001 C CNN
+F 0 "#PWR03" H 6400 4250 30  0001 C CNN
 F 1 "GND" H 6400 4180 30  0001 C CNN
 	1    6400 4250
@@
 $EndComp
 $Comp
-L R R2
-U 1 1 538370E5
-P 10850 6550
-F 0 "R2" V 10930 6550 50  0000 C CNN
-F 1 "10 kΩ" V 10850 6550 50  0000 C CNN
-	1    10850 6550
-	1    0    0    -1
-$EndComp
-$Comp
-L GND #PWR02
+L GND #PWR04
 U 1 1 53812E12
 P 10100 2050
-F 0 "#PWR02" H 10100 2050 30  0001 C CNN
+F 0 "#PWR04" H 10100 2050 30  0001 C CNN
 F 1 "GND" H 10100 1980 30  0001 C CNN
 	1    10100 2050
@@
 $EndComp
 $Comp
-L VCC #PWR03
+L VCC #PWR05
 U 1 1 53812E09
 P 10100 1350
-F 0 "#PWR03" H 10100 1450 30  0001 C CNN
+F 0 "#PWR05" H 10100 1450 30  0001 C CNN
 F 1 "VCC" H 10100 1450 30  0000 C CNN
 	1    10100 1350
@@
 $EndComp
 $Comp
-L GND #PWR04
+L GND #PWR06
 U 1 1 5380A4FE
 P 2300 4600
-F 0 "#PWR04" H 2300 4600 30  0001 C CNN
+F 0 "#PWR06" H 2300 4600 30  0001 C CNN
 F 1 "GND" H 2300 4530 30  0001 C CNN
 	1    2300 4600
@@
 $EndComp
 $Comp
-L VCC #PWR05
+L VCC #PWR07
 U 1 1 5380A4F9
 P 2300 3950
-F 0 "#PWR05" H 2300 4050 30  0001 C CNN
+F 0 "#PWR07" H 2300 4050 30  0001 C CNN
 F 1 "VCC" H 2300 4050 30  0000 C CNN
 	1    2300 3950
@@
 $EndComp
 $Comp
-L VCC #PWR06
+L VCC #PWR08
 U 1 1 5380A110
 P 950 1700
-F 0 "#PWR06" H 950 1800 30  0001 C CNN
+F 0 "#PWR08" H 950 1800 30  0001 C CNN
 F 1 "VCC" H 950 1800 30  0000 C CNN
 	1    950  1700
@@
 $EndComp
 $Comp
-L GND #PWR07
+L GND #PWR09
 U 1 1 5380A10C
 P 700 1850
-F 0 "#PWR07" H 700 1850 30  0001 C CNN
+F 0 "#PWR09" H 700 1850 30  0001 C CNN
 F 1 "GND" H 700 1780 30  0001 C CNN
 	1    700  1850
@@
 $EndComp
 $Comp
-L GND #PWR08
+L GND #PWR010
 U 1 1 5380A0B5
-P 2500 1700
-F 0 "#PWR08" H 2500 1700 30  0001 C CNN
-F 1 "GND" H 2500 1630 30  0001 C CNN
-	1    2500 1700
-	1    0    0    -1
-$EndComp
-$Comp
-L VCC #PWR09
+P 2500 2150
+F 0 "#PWR010" H 2500 2150 30  0001 C CNN
+F 1 "GND" H 2500 2080 30  0001 C CNN
+	1    2500 2150
+	-1   0    0    1
+$EndComp
+$Comp
+L VCC #PWR011
 U 1 1 5380A0B1
 P 2400 1700
-F 0 "#PWR09" H 2400 1800 30  0001 C CNN
+F 0 "#PWR011" H 2400 1800 30  0001 C CNN
 F 1 "VCC" H 2400 1800 30  0000 C CNN
 	1    2400 1700
@@
 $EndComp
 $Comp
-L VDD #PWR010
+L VDD #PWR012
 U 1 1 53809F25
 P 10750 3300
-F 0 "#PWR010" H 10750 3400 30  0001 C CNN
+F 0 "#PWR012" H 10750 3400 30  0001 C CNN
 F 1 "VDD" H 10750 3410 30  0000 C CNN
 	1    10750 3300
@@
 $EndComp
 $Comp
-L VCC #PWR011
+L VCC #PWR013
 U 1 1 53809F21
 P 10750 3200
-F 0 "#PWR011" H 10750 3300 30  0001 C CNN
+F 0 "#PWR013" H 10750 3300 30  0001 C CNN
 F 1 "VCC" H 10750 3300 30  0000 C CNN
 	1    10750 3200
@@
 $EndComp
 $Comp
-L GND #PWR012
+L GND #PWR014
 U 1 1 53809F1D
 P 10550 3200
-F 0 "#PWR012" H 10550 3200 30  0001 C CNN
+F 0 "#PWR014" H 10550 3200 30  0001 C CNN
 F 1 "GND" H 10550 3130 30  0001 C CNN
 	1    10550 3200
@@
 $EndComp
 $Comp
-L VSS #PWR013
+L VSS #PWR015
 U 1 1 53809F1A
 P 10550 3300
-F 0 "#PWR013" H 10550 3300 30  0001 C CNN
+F 0 "#PWR015" H 10550 3300 30  0001 C CNN
 F 1 "VSS" H 10550 3230 30  0000 C CNN
 	1    10550 3300
@@
 	0    -1   -1   0
 $EndComp
-Text Label 10400 6950 0    60   ~ 0
-FINT
-$Comp
-L VCC #PWR014
-U 1 1 53809656
-P 10850 6250
-F 0 "#PWR014" H 10850 6350 30  0001 C CNN
-F 1 "VCC" H 10850 6350 30  0000 C CNN
-	1    10850 6250
-	1    0    0    -1
-$EndComp
-Entry Wire Line
-	9700 6850 9800 6950
 Text Label 9850 6800 0    60   ~ 0
 INT
@@
 	9700 6700 9800 6800
 $Comp
-L GND #PWR015
+L GND #PWR016
 U 1 1 538092CF
 P 8650 6050
-F 0 "#PWR015" H 8650 6050 30  0001 C CNN
+F 0 "#PWR016" H 8650 6050 30  0001 C CNN
 F 1 "GND" H 8650 5980 30  0001 C CNN
 	1    8650 6050
@@
 	9600 6450 9700 6550
 $Comp
-L VCC #PWR016
+L VCC #PWR017
 U 1 1 53809224
 P 9600 4950
-F 0 "#PWR016" H 9600 5050 30  0001 C CNN
+F 0 "#PWR017" H 9600 5050 30  0001 C CNN
 F 1 "VCC" H 9600 5050 30  0000 C CNN
 	1    9600 4950
@@
 P 9450 5650
 F 0 "U8" H 9450 5750 60  0000 C CNN
-F 1 "74LS109" H 9450 5550 60  0000 C CNN
+F 1 "74HC109" H 9450 5550 60  0000 C CNN
 	1    9450 5650
 	1    0    0    -1
@@
 $EndComp
 $Comp
-L VCC #PWR017
+L VCC #PWR018
 U 1 1 53808811
 P 4000 7150
-F 0 "#PWR017" H 4000 7250 30  0001 C CNN
+F 0 "#PWR018" H 4000 7250 30  0001 C CNN
 F 1 "VCC" H 4000 7250 30  0000 C CNN
 	1    4000 7150
@@
 $EndComp
 $Comp
-L GND #PWR018
+L GND #PWR019
 U 1 1 5380880E
 P 4200 7150
-F 0 "#PWR018" H 4200 7150 30  0001 C CNN
+F 0 "#PWR019" H 4200 7150 30  0001 C CNN
 F 1 "GND" H 4200 7080 30  0001 C CNN
 	1    4200 7150
@@
 $EndComp
 $Comp
-L VCC #PWR019
+L VCC #PWR020
 U 1 1 538086E8
 P 3150 6100
-F 0 "#PWR019" H 3150 6200 30  0001 C CNN
+F 0 "#PWR020" H 3150 6200 30  0001 C CNN
 F 1 "VCC" H 3150 6200 30  0000 C CNN
 	1    3150 6100
-	0    -1   -1   0
-$EndComp
-$Comp
-L GND #PWR020
-U 1 1 538086CF
-P 1550 6050
-F 0 "#PWR020" H 1550 6050 30  0001 C CNN
-F 1 "GND" H 1550 5980 30  0001 C CNN
-	1    1550 6050
-	0    1    1    0
-$EndComp
-$Comp
-L C C2
-U 1 1 538086AD
-P 1900 6350
-F 0 "C2" H 1950 6450 50  0000 L CNN
-F 1 "27 pF" H 1950 6250 50  0000 L CNN
-	1    1900 6350
-	0    -1   -1   0
-$EndComp
-$Comp
-L C C1
-U 1 1 538086A9
-P 1900 5750
-F 0 "C1" H 1950 5850 50  0000 L CNN
-F 1 "27 pF" H 1950 5650 50  0000 L CNN
-	1    1900 5750
-	0    -1   -1   0
-$EndComp
-$Comp
-L CRYSTAL X1
-U 1 1 5380869F
-P 2300 6050
-F 0 "X1" H 2300 6200 60  0000 C CNN
-F 1 "CRYSTAL" H 2300 5900 60  0000 C CNN
-	1    2300 6050
 	0    -1   -1   0
 $EndComp
@@
 Entry Wire Line
 	6150 1750 6250 1850
-$Comp
-L 74LS374 U5
-U 1 1 537FA36C
-P 7100 1450
-F 0 "U5" H 7100 1450 60  0000 C CNN
-F 1 "74LS374" H 7150 1100 60  0000 C CNN
-	1    7100 1450
-	1    0    0    -1
-$EndComp
 Text Label 4700 1150 0    60   ~ 0
 IN_ENABLE
@@
 P 7100 3400
 F 0 "U6" H 7100 3400 60  0000 C CNN
-F 1 "74LS374" H 7150 3050 60  0000 C CNN
+F 1 "74HC374" H 7150 3050 60  0000 C CNN
 	1    7100 3400
 	1    0    0    -1
@@
 P 3950 1550
 F 0 "U2" H 3950 2450 60  0000 C CNN
-F 1 "74LS154" H 3900 700 60  0000 C CNN
+F 1 "74HC154" H 3900 700 60  0000 C CNN
 	1    3950 1550
 	1    0    0    -1
